File: Dragon32Rev3.5.kicad_pcb (KiCad board)
At the start: 2 copper layers, 253 x 199.4 mm, 129 parts, among them IC1 MC6809E, IC11 6551, IC2 MC6821, IC25 LM393P, IC3 74LS244N, IC34 CD4050BDR, IC35 MC6821, IC4 MC14529B, J1 DataBus, J10 RGBS Interface, J11 External Serial, J2 Video, J3 AddressBus, J4 ControlOut, J5 ControlIn, J6 Video_In, J7 BusService, J9 Video_Out, Q1 SS8050, SW1 RESET, U1 74AHCT1G08, U10 74LVC1G3157, U11 74LVC1G3157, U12 74LVC1G3157, U13 74LVC1G3157, U14 74LVC1G66DSF, U15 74LVC1G66DSF, U16 SLG46824V, U17 CD4077, U18 MAX3232, U19 28C256, U2 74ALS138N, U3 74ALS138N, U4 74ALS138N, U5 74ALS02, U6 74LVC1G3157, U7 74LVC1G3157, U8 74LVC1G3157, U9 74LVC1G3157

Commit message: add audio support
Parts:
- added C18: 10uF, Capacitor_SMD:CP_Elec_4x3, F.Cu at (246.0, 158.7)
- added C19: 10uF, Capacitor_SMD:CP_Elec_4x3, F.Cu at (251.8, 158.7)
- added C22: 10uF, Capacitor_SMD:CP_Elec_4x3, F.Cu at (144.1, 104.1)
- added C23: 10uF, Capacitor_SMD:CP_Elec_4x3, F.Cu at (156.2, 97.8)
- added C25: 10uF, Capacitor_SMD:CP_Elec_4x3, F.Cu at (146.9, 91.9)
- added C29: 10uF, Capacitor_SMD:CP_Elec_4x3, F.Cu at (146.9, 97.0)
- added IC38: 74LS08, Package_SO:SOIC-14_3.9x8.7mm_P1.27mm, F.Cu at (253.0, 216.3)
- added IC39: 74LS04, Package_SO:SOIC-14_3.9x8.7mm_P1.27mm, F.Cu at (263.1, 216.3)
- added IC5: AY-3-8910, Package_DIP:DIP-40_W15.24mm_Socket, F.Cu at (179.9, 172.8)
- added IC6: AY-3-8910, Package_DIP:DIP-40_W15.24mm_Socket, F.Cu at (209.5, 172.8)
- added IC7: AY-3-8912, Package_DIP:DIP-28_W15.24mm_Socket, F.Cu at (183.2, 180.4)
- added IC8: AY-3-8912, Package_DIP:DIP-28_W15.24mm_Socket, F.Cu at (212.9, 180.4)
- added J12: Stereo Audio, Connector_JST:JST_EH_S4B-EH_1x04_P2.50mm_Horizontal, F.Cu at (103.0, 66.4)
- added J8: AudioOut, Connector_PinHeader_2.54mm:PinHeader_1x08_P2.54mm_Vertical, F.Cu at (163.4, 106.1)
- added R18: 2.2K, PCM_Resistor_SMD_AKL:R_0603_1608Metric, F.Cu at (241.3, 164.5)
- added R19: 4K, PCM_Resistor_SMD_AKL:R_0603_1608Metric, F.Cu at (250.8, 164.5)
- added R20: 2.2K, PCM_Resistor_SMD_AKL:R_0603_1608Metric, F.Cu at (252.7, 164.5)
- added R21: 2.2K, PCM_Resistor_SMD_AKL:R_0603_1608Metric, F.Cu at (243.2, 164.5)
- added R22: 4K, PCM_Resistor_SMD_AKL:R_0603_1608Metric, F.Cu at (245.2, 164.5)
- added R23: 2.2K, PCM_Resistor_SMD_AKL:R_0603_1608Metric, F.Cu at (254.5, 164.5)
- added R24: 1K, PCM_Resistor_SMD_AKL:R_0603_1608Metric, F.Cu at (240.5, 160.7)
- added R25: 1K, PCM_Resistor_SMD_AKL:R_0603_1608Metric, F.Cu at (257.2, 160.7)
- added R26: 4K, PCM_Resistor_SMD_AKL:R_0603_1608Metric, F.Cu at (247.1, 164.5)
- added R27: 4K, PCM_Resistor_SMD_AKL:R_0603_1608Metric, F.Cu at (256.3, 164.5)
- added RN4: 22R, PCM_Resistor_SMD_AKL:R_Array_Convex_4x0603, F.Cu at (156.5, 106.8)
- added U20: 74LS93, Package_SO:SOIC-14_3.9x8.7mm_P1.27mm, F.Cu at (242.9, 216.3)
- added U21: PCM1754DBQ, Package_SO:SSOP-16_3.9x4.9mm_P0.635mm, F.Cu at (150.4, 104.0)
- J2: footprint Connector_PinHeader_2.54mm:PinHeader_1x07_P2.54mm_Vertical -> Connector_PinHeader_2.54mm:PinHeader_1x08_P2.54mm_Vertical
- moved RV3 4.06 mm to (65.6, 99.8)
- moved C35 2.01 mm to (133.3, 110.2)
- moved R46 1.16 mm to (136.9, 103.8), turned to -90 degrees
- moved C44 1.10 mm to (136.9, 107.2), turned to 90 degrees
Connections:
- net /Devices/A0 renamed /Audio/A0
- net /Devices/A1 renamed /Audio/A1
- net /Devices/A10 renamed /Audio/A10
- net /Devices/A11 renamed /Audio/A11
- net /Devices/A12 renamed /Audio/A12
- net /Devices/A13 renamed /Audio/A13
- net /Devices/A14 renamed /Audio/A14
- net /Devices/A15 renamed /Audio/A15
- net /Devices/A2 renamed /Audio/A2
- net /Devices/A3 renamed /Audio/A3
- net /Devices/A4 renamed /Audio/A4
- net /Devices/A5 renamed /Audio/A5
- net /Devices/A6 renamed /Audio/A6
- net /Devices/A7 renamed /Audio/A7
- net /Devices/A9 renamed /Audio/A9
- net /Devices/D0 renamed /Audio/D0
- net /Devices/D1 renamed /Audio/D1
- net /Devices/D2 renamed /Audio/D2
- net /Devices/D3 renamed /Audio/D3
- net /Devices/D4 renamed /Audio/D4
- net /Devices/D5 renamed /Audio/D5
- net /Devices/D6 renamed /Audio/D6
- net /Devices/D7 renamed /Audio/D7
- IC1 pad 16: /Devices/A8 -> /Audio/A8
- J3 pad 9: /Devices/A8 -> /Audio/A8
- PL7 pad 27: /Devices/A8 -> /Audio/A8
- U19 pad 25: /Devices/A8 -> +5V
Routing:
- net SOUND B: track 0.00 -> 308.3 mm, vias 0 -> 2
- net +5V: track 1398.0 -> 1683.6 mm, vias 50 -> 53
- net SOUND A: track 0.00 -> 238.9 mm, vias 0 -> 2
- net SP13: track 0.00 -> 234.3 mm, vias 0 -> 2
- net SP12: track 0.00 -> 213.3 mm, vias 0 -> 2
- net VCLK: track 0.00 -> 206.2 mm, vias 0 -> 3
- net /Audio/D0: track 341.9 -> 494.7 mm, vias 2 -> 4
- net /Audio/A8: track 0.00 -> 151.2 mm, vias 0 -> 2
- net /Devices/A8: track 151.2 -> 0.00 mm, vias 2 -> 0
- net /Audio/D1: track 339.6 -> 488.7 mm, vias 2 -> 5
- net /Audio/D2: track 348.4 -> 491.5 mm, vias 2 -> 5
- net /Audio/D3: track 329.7 -> 467.9 mm, vias 2 -> 5
- net /Audio/D4: track 337.7 -> 468.5 mm, vias 2 -> 5
- net /Audio/D5: track 334.7 -> 459.8 mm, vias 2 -> 5
- net /Audio/D6: track 342.9 -> 463.2 mm, vias 2 -> 5
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